Commit message: robot urdf modeling

File: src/robot/robot_arm.urdf (robot description, URDF)
Before this commit: robot 3dof_robot_arm, 5 links, 4 joints
Links:
- removed link base_link
- removed link end_effector
- removed link link1
- removed link link2
- removed link link3
- added link Base, mass 1.0; collision box size=0.10 0.10 0.01; visual box size=0.10 0.10 0.01
- added link Body, mass 0.5; collision cylinder length=0.085 radius=0.0325; visual cylinder length=0.085 radius=0.0325
- added link End Effector, mass 0.1; collision box size=0.05 0.01 0.01; visual box size=0.05 0.01 0.01
- added link Forearm, mass 0.3; collision box size=0.17 0.02 0.02; visual box size=0.17 0.02 0.02
- added link UpperArm, mass 0.3; collision box size=0.16 0.02 0.02; visual box size=0.16 0.02 0.02
Joints:
- removed joint base_to_link1
- removed joint link1_to_link2
- removed joint link2_to_link3
- removed joint link3_to_end_effector
- added joint Elbow: type revolute, parent UpperArm, child Forearm, origin xyz=0.16 0 0 rpy=0 0 0, axis 0 1 0, limit lower=0.087 upper=3.14 effort=100 velocity=1.0
- added joint Rotator: type revolute, parent Base, child Body, origin xyz=0 0 0.005 rpy=0 0 0, axis 0 0 1, limit lower=-3.14 upper=3.14 effort=100 velocity=1.0
- added joint Shoulder: type revolute, parent Body, child UpperArm, origin xyz=0 0 0.085 rpy=0 0 0, axis 0 1 0, limit lower=-2.09 upper=0.52 effort=100 velocity=1.0
- added joint Wrist: type revolute, parent Forearm, child End Effector, origin xyz=0.17 0 0 rpy=0 0 0, axis 0 1 0, limit lower=-1.57 upper=1.57 effort=100 velocity=1.0

Commit message: URDF aligned with TF broadcast. calibration still needed

File: src/robot/robot_arm.urdf (robot description, URDF)
Before this commit: robot 3dof_robot_arm, 5 links, 4 joints
Links:
- removed link Forearm
- removed link UpperArm
- added link Fore Arm, mass 0.3; collision box size=0.17 0.02 0.02; visual box size=0.17 0.02 0.02
- added link Upper Arm, mass 0.3; collision box size=0.16 0.02 0.02; visual box size=0.16 0.02 0.02
Joints:
- joint Elbow: child Forearm -> Fore Arm; parent UpperArm -> Upper Arm
- joint Shoulder: child UpperArm -> Upper Arm
- joint Wrist: parent Forearm -> Fore Arm

Commit message: modified range in urdf rotator joint

File: src/robot/robot_arm.urdf (robot description, URDF)
Before this commit: robot 3dof_robot_arm, 5 links, 4 joints
Joints:
- joint Rotator: limit lower=-3.14 upper=3.14 effort=100 velocity=1.0 -> lower=-0.785398 upper=0.785398 effort=100 velocity=1.0
